File: STM32-DevBoard.kicad_sch (KiCad schematic)
At the start: 56 parts, among them J1 Conn_01x08_Pin, J2 I2C Bus 1, J3 Serial Debugger, J4 USART1, J5 12402012E212A, J6 PJ-002A, Q1 AO3401A, SW1 SW_SPDT, U1 STM32F103C8T6, U2 TPS563209DDCR, U3 USBLC6-2SC6, Y1 16MHz

Commit message: Completed net names
Connections:
- net SW_OUT: now reaches C14.1, L1.1, U2.2 (SW)
- net VBST_OUT: now reaches C14.2, U2.6 (VBST)
- net USB_DN: now reaches R4.1, U1.32 (PA11)
- net CC1_B: now reaches J5.B5 (CC1_B), R10.1
- net VIN_FUSED: now reaches F1.2, FB1.1
- net VFB_OUT: now reaches R8.2, R9.1, U2.4 (VFB)
- net USB_DP: now reaches R5.1, U1.33 (PA12)
- net LED2: now reaches D3.2 (A), U1.12 (PA2)
- net VIN_PROTECTED: now reaches D1.1 (K), F1.1, Q1.2 (S)
- net CC1_A: now reaches J5.A5 (CC1_A), R12.1
- net LED1: now reaches D2.2 (A), U1.11 (PA1)
- net DP_AB: now reaches J5.A6 (D+_A), J5.B6 (D+_B), U3.1 (I/O1)
- net DN_AB: now reaches J5.A7 (D-_A), J5.B7 (D-_B), U3.3 (I/O2)
- no-connect marks 22 -> 21
Other:
- moved on the sheet: C14, C18, C19, D1, F1, FB1, Q1, R13, R4, R5, U3

Commit message: Routing progressed
Parts:
- D4: value LED1 -> PLED
- J1: footprint Connector_PinHeader_1.00mm:PinHeader_1x08_P1.00mm_Vertical -> Connector_PinHeader_2.00mm:PinHeader_1x08_P2.00mm_Vertical
Connections:
- net DN_AB is gone; now on net USB_D-: J5.A7 (D-_A), J5.B7 (D-_B), U3.3 (I/O2)
- net DP_AB is gone; now on net USB_D+: J5.A6 (D+_A), J5.B6 (D+_B), U3.1 (I/O1)
- net USB_D+: now also U1.33 (PA12); no longer R5.2
- net USB_D-: now also U1.32 (PA11); no longer R4.2
- net LED1-: now reaches D2.1 (K), R6.1
- net LED2-: now reaches D3.1 (K), R7.1
- net PLED_OUT: now reaches D4.1 (K), R11.2
- net LED1 renamed LED1+
- net LED2 renamed LED2+
- net USB_DN: no longer names the net of R4.1
- net USB_DN: no longer U1.32 (PA11)
- net USB_DP: no longer names the net of R5.1
- net USB_DP: no longer U1.33 (PA12)
Other:
- moved on the sheet: D4, R4, R5, R6, R7
