File: STM32-DevBoard.kicad_sch (KiCad schematic)
At the start: 56 parts, among them J1 Conn_01x08_Pin, J2 I2C Bus 1, J3 Serial Debugger, J4 USART1, J5 12402012E212A, J6 PJ-002A, Q1 AO3401A, SW1 SW_SPDT, U1 STM32F103C8T6, U2 TPS563209DDCR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

Commit message: Net labels partially complete, still more to go
Connections:
- net USB_D+: no longer R4.2, U3.6 (I/O1)
- new net USB_D-: R4.2, U3.6 (I/O1)
Changed lines of the file:
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@@
+		)
+	)
+	(label "USBF_D+"
+		(at 262.89 100.33 0)
+		(effects
+			(font
+				(size 1.27 1.27)
+			)
+			(justify left bottom)
 		)
 	)
@@
 		)
 	)
-	(label "USB_D-"
-		(at 262.89 102.87 0)
-		(effects
-			(font
-				(size 1.27 1.27)
-			)
-			(justify left bottom)
-		)
-	)
 	(label "HSE_IN"
 		(at 64.77 119.38 0)
@@
 		)
 	)
+	(label "USBF_D-"
+		(at 262.89 102.87 0)
+		(effects
+			(font
+				(size 1.27 1.27)
+			)
+			(justify left bottom)
+		)
+	)
 	(label "VFB_OUT"
 		(at 165.1 43.18 0)
-		(effects
-			(font
-				(size 1.27 1.27)
-			)
-			(justify left bottom)
-		)
-	)
-	(label "USB_D+"
-		(at 262.89 100.33 0)
 		(effects
 			(font
@@
 			)
 		)
+	)
+	(netclass_flag ""
+		(length 2.54)
+		(shape round)
+		(at 24.13 88.9 0)
+		(fields_autoplaced yes)
+		(effects
+			(font
+				(size 1.27 1.27)
+			)
+			(justify left bottom)
+		)
+		(property "Netclass" "Power"
+			(at 24.8285 86.36 0)
+			(effects
+				(font
+					(size 1.27 1.27)
+				)
+				(justify left)
+			)
+		)
+		(property "Component Class" ""
+			(at -264.16 30.48 0)
+			(effects
+				(font
+					(size 1.27 1.27)
+					(italic yes)
+				)
+			)
+		)
+	)
+	(netclass_flag ""
+		(length 2.54)
+		(shape round)
+		(at 105.41 54.61 0)
+		(fields_autoplaced yes)
+		(effects
+			(font
+				(size 1.27 1.27)
+			)
+			(justify left bottom)
+		)
+		(property "Netclass" "GND"
+			(at 106.1085 52.07 0)
+			(effects
+				(font
+					(size 1.27 1.27)
+				)
+				(justify left)
+			)
+		)
+		(property "Component Class" ""
+			(at -55.88 -43.18 0)
+			(effects
+				(font
+					(size 1.27 1.27)
+					(italic yes)
+				)
+			)
+		)
